File: his_masters_noise.sch (EAGLE design)
At the start: 39 parts, among them IC1 TL074P, IC2 NE555N, IC3 40106N, IC4 4013N, T1 2N3904, T2 2N3904

Commit message: digital noise
Parts:
- renumbered PINKISH_NOISE1 to DIGITAL_NOISE
Changed lines of the file:
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@@
 <part name="C8" library="rcl" library_urn="urn:adsk.eagle:library:334" deviceset="CPOL-EU" device="E1.8-4" package3d_urn="urn:adsk.eagle:package:23336/2" value="2.2uF"/>
 <part name="GND15" library="supply1" library_urn="urn:adsk.eagle:library:371" deviceset="GND" device=""/>
-<part name="PINKISH_NOISE1" library="thonkiconn" deviceset="WQP-PJ301M-12_JACK" device=""/>
+<part name="DIGITAL_NOISE" library="thonkiconn" deviceset="WQP-PJ301M-12_JACK" device=""/>
 <part name="GND16" library="supply1" library_urn="urn:adsk.eagle:library:371" deviceset="GND" device=""/>
 <part name="GND17" library="supply1" library_urn="urn:adsk.eagle:library:371" deviceset="GND" device=""/>
@@
 <attribute name="VALUE" x="-38.1" y="403.86" size="1.778" layer="96"/>
 </instance>
-<instance part="PINKISH_NOISE1" gate="G$1" x="170.18" y="401.32" smashed="yes">
+<instance part="DIGITAL_NOISE" gate="G$1" x="170.18" y="401.32" smashed="yes">
 <attribute name="NAME" x="167.64" y="405.384" size="1.778" layer="95"/>
 </instance>
@@
 <segment>
 <pinref part="IC4" gate="A" pin="Q"/>
-<pinref part="PINKISH_NOISE1" gate="G$1" pin="2"/>
+<pinref part="DIGITAL_NOISE" gate="G$1" pin="2"/>
 <wire x1="157.48" y1="403.86" x2="165.1" y2="403.86" width="0.1524" layer="91"/>
 </segment>
